File: RFLED/RFLED.brd (EAGLE design)
At the start: 63.2 x 26.7 mm, 6 parts

Commit message: More tedious updates.
Parts:
- removed TCS3472: TC3472DFNL6_WIDE, DZ:DFNL6_WIDE
- removed U$1: AUDIO-JACK3, SparkFun-Connectors:AUDIO-JACK-TRRS-SMD
- added C1, C2: 0.1uF, SparkFun-Capacitors:0603-CAP
- added J3: AUDIO-JACK3, SparkFun-Connectors:AUDIO-JACK-TRRS-SMD
- added U10: TC3472DFNL6_WIDE, DZ:DFNL6_WIDE
- added U3: (no value), SparkFun-PowerIC:SOT23-5
- renumbered RFM12B to U1, U$2 to J1, U$3 to J2, WS8201-1 to U2
Connections:
- removed net J_GND: TCS3472.GND, U$1.EARTH
- new net N$1: J3.EARTH, U3.1
- new net N$2: U10.VDD
- net J_SCL: now also J3.TIP, U10.SCL; no longer TCS3472.SCL, U$1.TIP
- net J_SDA: now also J3.RING1, U10.SDA; no longer TCS3472.SDA, U$1.RING1
- net J_VDD: now also J3.RING2; no longer TCS3472.VDD, U$1.RING2
- net VDD: no longer J2.RING2
Routing:
- net J_SCL: track 0.00 -> 8.95 mm, vias 0 -> 1
Changed lines of the file:
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@@
 </autorouter>
 <elements>
-<element name="RFM12B" library="JeeParts" package="RFM12B" value="RFM12B" x="43.18" y="8.89" rot="R180"/>
-<element name="TCS3472" library="DZ" package="DFNL6_WIDE" value="TC3472DFNL6_WIDE" x="3.81" y="8.89" rot="MR270"/>
-<element name="U$2" library="DZ" package="TRINKET_SHIELD" value="TRINKET_SHIELD" x="24.13" y="10.16" rot="R90"/>
-<element name="WS8201-1" library="SparkFun-DigitalIC" package="SOP-14" value="WS2801" x="27.94" y="8.89"/>
-<element name="U$1" library="SparkFun-Connectors" package="AUDIO-JACK-TRRS-SMD" value="AUDIO-JACK3" x="3.81" y="0" rot="R90"/>
-<element name="U$3" library="SparkFun-Connectors" package="AUDIO-JACK-TRRS-SMD" value="AUDIO-JACK3" x="16.51" y="0" rot="R90"/>
+<element name="U1" library="JeeParts" package="RFM12B" value="RFM12B" x="43.18" y="8.89" rot="R180"/>
+<element name="J1" library="DZ" package="TRINKET_SHIELD" value="TRINKET_SHIELD" x="24.13" y="10.16" rot="R90"/>
+<element name="U2" library="SparkFun-DigitalIC" package="SOP-14" value="WS2801" x="27.94" y="8.89"/>
+<element name="J3" library="SparkFun-Connectors" package="AUDIO-JACK-TRRS-SMD" value="AUDIO-JACK3" x="5.08" y="0" rot="R90"/>
+<element name="J2" library="SparkFun-Connectors" package="AUDIO-JACK-TRRS-SMD" value="AUDIO-JACK3" x="16.51" y="0" rot="R90"/>
+<element name="U10" library="DZ" package="DFNL6_WIDE" value="TC3472DFNL6_WIDE" x="7.62" y="5.08" rot="MR270"/>
+<element name="U3" library="SparkFun-PowerIC" package="SOT23-5" value="" x="-2.54" y="0">
+<attribute name="PROD_ID" value="VREG-00822" x="-2.54" y="0" size="1.778" layer="27" display="off"/>
+</element>
+<element name="C1" library="SparkFun-Capacitors" package="0603-CAP" value="0.1uF" x="-2.54" y="-3.81">
+<attribute name="PROD_ID" value="CAP-00810" x="-2.54" y="-3.81" size="1.778" layer="27" display="off"/>
+</element>
+<element name="C2" library="SparkFun-Capacitors" package="0603-CAP" value="0.1uF" x="-2.54" y="-7.62">
+<attribute name="PROD_ID" value="CAP-00810" x="-2.54" y="-7.62" size="1.778" layer="27" display="off"/>
+</element>
 </elements>
 <signals>
 <signal name="BAT+">
-<contactref element="U$2" pad="BAT+"/>
+<contactref element="J1" pad="BAT+"/>
 </signal>
 <signal name="VBUS">
-<contactref element="U$2" pad="USB+"/>
+<contactref element="J1" pad="USB+"/>
 </signal>
 <signal name="GND">
-<contactref element="U$2" pad="GND"/>
-<contactref element="RFM12B" pad="GND"/>
-<contactref element="WS8201-1" pad="7"/>
-<contactref element="U$3" pad="EARTH"/>
-<wire x1="22.86" y1="2.54" x2="35.18" y2="10.89" width="0" layer="19" extent="1-1"/>
+<contactref element="J1" pad="GND"/>
+<contactref element="U1" pad="GND"/>
+<contactref element="U2" pad="7"/>
+<contactref element="J2" pad="EARTH"/>
 <wire x1="31.75" y1="6.14" x2="35.18" y2="10.89" width="0" layer="19" extent="1-1"/>
+<wire x1="22.86" y1="2.54" x2="31.75" y2="6.14" width="0" layer="19" extent="1-1"/>
 <wire x1="19.76" y1="11.3" x2="22.86" y2="2.54" width="0" layer="19" extent="1-1"/>
 </signal>
 <signal name="SDA">
-<contactref element="U$2" pad="#0"/>
-<contactref element="WS8201-1" pad="2"/>
-<contactref element="U$3" pad="RING1"/>
+<contactref element="J1" pad="#0"/>
+<contactref element="U2" pad="2"/>
+<contactref element="J2" pad="RING1"/>
 <wire x1="25.4" y1="6.14" x2="22.86" y2="15.24" width="0" layer="19" extent="1-1"/>
 <wire x1="13.26" y1="6.2" x2="25.4" y2="6.14" width="0" layer="19" extent="1-1"/>
 </signal>
 <signal name="MISO">
-<contactref element="U$2" pad="#1"/>
-<contactref element="RFM12B" pad="SDI"/>
+<contactref element="J1" pad="#1"/>
+<contactref element="U1" pad="SDI"/>
 <wire x1="35.18" y1="6.89" x2="25.4" y2="15.24" width="0" layer="19" extent="1-1"/>
 </signal>
 <signal name="SCL">
-<contactref element="U$2" pad="#2"/>
-<contactref element="WS8201-1" pad="1"/>
-<contactref element="U$3" pad="TIP"/>
+<contactref element="J1" pad="#2"/>
+<contactref element="U2" pad="1"/>
+<contactref element="J2" pad="TIP"/>
 <wire x1="24.13" y1="6.14" x2="27.94" y2="15.24" width="0" layer="19" extent="1-1"/>
 <wire x1="13.26" y1="10.2" x2="24.13" y2="6.14" width="0" layer="19" extent="1-1"/>
 </signal>
 <signal name="MOSI">
-<contactref element="U$2" pad="#3"/>
-<contactref element="RFM12B" pad="SDO"/>
+<contactref element="J1" pad="#3"/>
+<contactref element="U1" pad="SDO"/>
 <wire x1="27.94" y1="2.54" x2="51.18" y2="2.89" width="0" layer="19" extent="1-1"/>
 </signal>
 <signal name="CLK">
-<contactref element="U$2" pad="#4"/>
-<contactref element="RFM12B" pad="SCK"/>
+<contactref element="J1" pad="#4"/>
+<contactref element="U1" pad="SCK"/>
 <wire x1="25.4" y1="2.54" x2="35.18" y2="4.89" width="0" layer="19" extent="1-1"/>
 </signal>
 <signal name="VDD">
-<contactref element="RFM12B" pad="SEL"/>
-<contactref element="RFM12B" pad="VDD"/>
-<contactref element="U$2" pad="3V"/>
-<contactref element="WS8201-1" pad="14"/>
-<contactref element="U$3" pad="RING2"/>
+<contactref element="U1" pad="SEL"/>
+<contactref element="U1" pad="VDD"/>
+<contactref element="J1" pad="3V"/>
+<contactref element="U2" pad="14"/>
 <wire x1="30.48" y1="15.24" x2="35.18" y2="12.89" width="0" layer="19" extent="1-1"/>
+<wire x1="24.13" y1="11.64" x2="30.48" y2="15.24" width="0" layer="19" extent="1-1"/>
 <wire x1="35.18" y1="2.89" x2="35.18" y2="12.89" width="0" layer="19" extent="1-1"/>
-<wire x1="24.13" y1="11.64" x2="30.48" y2="15.24" width="0" layer="19" extent="1-1"/>
-<wire x1="13.26" y1="3.2" x2="24.13" y2="11.64" width="0" layer="19" extent="1-1"/>
-</signal>
-<signal name="J_GND">
-<contactref element="U$1" pad="EARTH"/>
-<contactref element="TCS3472" pad="GND"/>
-<wire x1="4.46" y1="9.69" x2="7.06" y2="11.3" width="0" layer="19" extent="1-1"/>
 </signal>
 <signal name="J_VDD">
-<contactref element="TCS3472" pad="VDD"/>
-<contactref element="U$1" pad="RING2"/>
-<wire x1="3.16" y1="9.69" x2="0.56" y2="3.2" width="0" layer="19" extent="1-1"/>
+<contactref element="J3" pad="RING2"/>
 </signal>
 <signal name="J_SDA">
-<contactref element="U$1" pad="RING1"/>
-<contactref element="TCS3472" pad="SDA"/>
-<wire x1="3.16" y1="8.14" x2="0.56" y2="6.2" width="0" layer="19" extent="1-1"/>
+<contactref element="J3" pad="RING1"/>
+<contactref element="U10" pad="SDA"/>
+<wire x1="6.97" y1="4.33" x2="1.83" y2="6.2" width="0" layer="19" extent="1-1"/>
 </signal>
 <signal name="J_SCL">
-<contactref element="U$1" pad="TIP"/>
-<contactref element="TCS3472" pad="SCL"/>
-<wire x1="0.56" y1="10.2" x2="3.81" y2="9.69" width="0" layer="19" extent="1-1"/>
+<contactref element="J3" pad="TIP"/>
+<contactref element="U10" pad="SCL"/>
+<wire x1="1.83" y1="10.2" x2="1.83" y2="9.6" width="0.4064" layer="1"/>
+<wire x1="1.83" y1="9.6" x2="3.81" y2="7.62" width="0.4064" layer="1"/>
+<wire x1="3.81" y1="7.62" x2="6.35" y2="7.62" width="0.4064" layer="1"/>
+<via x="6.35" y="7.62" extent="1-16" drill="0.6"/>
+<wire x1="7.62" y1="5.88" x2="7.62" y2="7.62" width="0.4064" layer="16"/>
+<wire x1="7.62" y1="7.62" x2="6.35" y2="7.62" width="0.4064" layer="16"/>
+</signal>
+<signal name="N$2">
+<contactref element="U10" pad="VDD"/>
+</signal>
+<signal name="N$1">
+<contactref element="J3" pad="EARTH"/>
+<contactref element="U3" pad="1"/>
+<wire x1="-3.49" y1="-1.3001" x2="8.33" y2="11.3" width="0" layer="19" extent="1-1"/>
 </signal>
 </signals>
