File: RFLED/RFLED.sch (EAGLE design)
At the start: 6 parts

Commit message: More tedious updates.
Parts:
- removed TCS3472: TC3472DFNL6_WIDE, DZ:TC3472DFNL6_WIDE
- removed U$1, U$3: AUDIO-JACK3, SparkFun-Connectors:AUDIO-JACK3
- added C1, C2: 0.1uF, SparkFun-Capacitors:0.1UF-25V(+80/-20%)(0603)
- added J2, J3: AUDIO-JACK3, SparkFun-Connectors:AUDIO-JACK3
- added U10: TC3472DFNL6_WIDE, DZ:TC3472DFNL6_WIDE
- added U3: (no value), SparkFun-PowerIC:MIC52053.3V
- renumbered RFM12B to U1, U$2 to J1, WS8201-1 to U2
Connections:
- removed net J_GND: TCS3472.GND, U$1.EARTH
- new net N$1: J3.EARTH, U3.IN
- new net N$2: U10.VDD
- net GND: now also J2.EARTH; no longer U$3.EARTH
- net J_SCL: now also J3.TIP, U10.SCL; no longer TCS3472.SCL, U$1.TIP
- net J_SDA: now also J3.RING1, U10.SDA; no longer TCS3472.SDA, U$1.RING1
- net J_VDD: now also J3.RING2; no longer TCS3472.VDD, U$1.RING2
- net SCL: now also J2.TIP; no longer U$3.TIP
- net SDA: now also J2.RING1; no longer U$3.RING1
- net VDD: no longer U$3.RING2
